Commit message: robot with kinect

File: urdf/udacity_bot.xacro (robot description, xacro)
@@ -146,31 +146,44 @@
   </joint>
 <!--CAMERA-->
- <link name="camera">
-   <inertial>
-     <origin xyz="0.0 0.0 0.0" rpy="0.0 0.0 0.0"/>
-     <mass value="0.1"/>
-      <inertia ixx="1e-6" ixy="0" ixz="0" iyy="1e-6" iyz="0" izz="1e-6"/>
-    </inertial>
-   <visual>
-     <origin xyz="0.0 0.0 0.0" rpy="0.0 0.0 0.0"/>
-     <geometry>
-       <box size=".05 .05 .05"/>
-     </geometry>
-   </visual>
-   <collision>
-     <origin xyz="0.0 0.0 0.0" rpy="0.0 0.0 0.0"/>
-     <geometry>
-       <box size=".05 .05 .05"/>
-     </geometry>
-   </collision>
- </link>
-  <joint type="fixed" name="camera_joint">
-    <origin xyz="0.2 0.0 0.0" rpy="0 0 0"/>
-    <child link="camera"/>
-    <parent link="chassis"/>
-    <axis xyz="0 1 0" rpy="0 0 0"/>
-    <limit effort="10000" velocity="1000"/>
-    <joint_properties damping="1.0" friction="1.0"/>
-  </joint>
+<link name="camera">
+ <inertial>
+   <origin xyz="0.0 0.0 0.0" rpy="0.0 0.0 0.0"/>
+   <mass value="0.1"/>
+    <inertia ixx="1e-6" ixy="0" ixz="0" iyy="1e-6" iyz="0" izz="1e-6"/>
+  </inertial>
+ <visual>
+   <origin xyz="0.0 0.0 0.0" rpy="0.0 0.0 0.0"/>
+   <geometry>
+   		<mesh filename="package://slam_project/meshes/kinect.dae"/>
+   </geometry>
+ </visual>
+ <collision>
+   <origin xyz="0.0 0.0 0.0" rpy="0.0 0.0 0.0"/>
+   <geometry>
+     <box size=".05 .05 .05"/>
+   </geometry>
+ </collision>
+</link>
+<joint type="fixed" name="camera_joint">
+  <origin xyz="0.3 0.0 0.0" rpy="0 0 0"/>
+  <child link="camera"/>
+  <parent link="chassis"/>
+  <axis xyz="0 1 0" rpy="0 0 0"/>
+  <limit effort="10000" velocity="1000"/>
+  <joint_properties damping="1.0" friction="1.0"/>
+</joint>
+<!-- RGBD camera -->
+<link name="rgbd_camera">
+ <inertial>
+   <origin xyz="0.0 0.0 0.0" rpy="0.0 0.0 0.0"/>
+   <mass value="0.0"/>
+   <inertia ixx="1e-6" ixy="0" ixz="0" iyy="1e-6" iyz="0" izz="1e-6"/>
+  </inertial>
+</link>
+<joint type="fixed" name="rgbd_joint">
+  <origin xyz="0.0 0.0 0.0" rpy="-1.5707 0 0"/>
+  <child link="rgbd_camera"/>
+  <parent link="camera"/>
+</joint>
 <!--LASER-->
 <link name="hokuyo">

Commit message: fix to joint rotation

File: urdf/udacity_bot.xacro (robot description, xacro)
@@ -2,4 +2,5 @@
 <robot name="udacity_bot" xmlns:xacro="http://www.ros.org/wiki/xacro">
   <xacro:include filename="$(find slam_project)/urdf/udacity_bot.gazebo" />
+  <xacro:property name="M_PI" value="3.1415926535897931" />
   <link name="robot_footprint"></link>
   <joint name="robot_footprint_joint" type="fixed">
@@ -182,5 +183,5 @@
 </link>
 <joint type="fixed" name="rgbd_joint">
-  <origin xyz="0.0 0.0 0.0" rpy="-1.5707 0 0"/>
+  <origin xyz="0.0 0.0 0.0" rpy="${-M_PI/2} 0 ${-M_PI/2}"/>
   <child link="rgbd_camera"/>
   <parent link="camera"/>
